File: IDP_Circuitry/IDP_Circuitry.kicad_pcb (KiCad board)
At the start: 0 parts

Commit message: added all footprints, added libraryIDP for flipped pin header schematic
Parts:
- added C1: 22u, Capacitor_THT:C_Radial_D5.0mm_H5.0mm_P2.00mm, F.Cu at (25.5, 75.5)
- added LineTracker1: Conn_01x03_Pin, Connector_PinSocket_2.54mm:PinSocket_1x03_P2.54mm_Vertical, F.Cu at (25.9, 3.08)
- added LineTracker2: Conn_01x03_Pin, Connector_PinSocket_2.54mm:PinSocket_1x03_P2.54mm_Vertical, F.Cu at (25.9, 11.0)
- added LineTracker3: Conn_01x03_Pin, Connector_PinSocket_2.54mm:PinSocket_1x03_P2.54mm_Vertical, F.Cu at (25.9, 18.9)
- added LineTracker4: Conn_01x03_Pin, Connector_PinSocket_2.54mm:PinSocket_1x03_P2.54mm_Vertical, F.Cu at (25.9, 26.8)
- added Pico_W1: RaspberryPi_Pico_W, Module:RaspberryPi_Pico_Common_THT, F.Cu at (144.2, 67.0)
- added PinoutL1: Conn_01x20, Connector_PinHeader_2.54mm:PinHeader_1x20_P2.54mm_Vertical, F.Cu at (116.0, 15.7)
- added PinoutR1: Conn_01x20, LibraryIDP:PinHeader_1x20_P2.54mm_Vertical_Flipped_21-40, F.Cu at (184.5, 14.5)
- added PushButton1: Conn_01x03_Pin, Connector_PinSocket_2.54mm:PinSocket_1x03_P2.54mm_Vertical, F.Cu at (25.9, 34.7)
- added R1: 68k, Resistor_THT:R_Axial_DIN0207_L6.3mm_D2.5mm_P2.54mm_Vertical, F.Cu at (41.0, 81.0)
- added SchmittTrigger1: CD4093BE, CD4093BE:DIP794W45P254L1969H508Q14, F.Cu at (38.5, 114.9)
- added UltrasonicDistanceSensor1: Conn_01x03_Pin, Connector_PinSocket_2.54mm:PinSocket_1x03_P2.54mm_Vertical, F.Cu at (62.5, 32.5)
- added YellowLED1: Conn_01x03_Pin, Connector_PinSocket_2.54mm:PinSocket_1x03_P2.54mm_Vertical, F.Cu at (38.9, 66.5)
Other:
- copper layers 0 -> 2
